File: BatterySource-Kicad/BatterySource-Kicad.kicad_sch (KiCad schematic)
At the start: 0 parts

Commit message: Playing in kicad
Parts:
- added D1, D2, D3: 1N4007, Diode_THT:D_DO-41_SOD81_P10.16mm_Horizontal, symbol Diode:1N4007
- added R1: 1k, symbol Device:R
Connections:
- new net: D1.2 (A), D2.1 (K)
- new net: D3.2 (A), R1.2
- new net: D2.2 (A), D3.1 (K)
- new net +12V: R1.1
- new net GND: D1.1 (K)
Changed lines of the file:
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@@
 (kicad_sch (version 20230121) (generator eeschema)
   (paper "A4")
-  (symbol_instances)
+  (wire (pts (xy 92.71 91.44) (xy 92.71 100.33))
+    (stroke (width 0) (type default))
+  )
+  (wire (pts (xy 92.71 40.64) (xy 92.71 50.8))
+    (stroke (width 0) (type default))
+  )
+  (wire (pts (xy 92.71 58.42) (xy 92.71 68.58))
+    (stroke (width 0) (type default))
+  )
+  (symbol (lib_id "Diode:1N4007") (at 92.71 87.63 90) (unit 1)
+    (in_bom yes) (on_board yes) (dnp no) (fields_autoplaced)
+    (property "Reference" "D1" (at 95.25 86.36 90)
+      (effects (font (size 1.27 1.27)) (justify right))
+    )
+    (property "Value" "1N4007" (at 95.25 88.9 90)
+      (effects (font (size 1.27 1.27)) (justify right))
+    )
+    (property "Footprint" "Diode_THT:D_DO-41_SOD81_P10.16mm_Horizontal" (at 97.155 87.63 0)
+      (effects (font (size 1.27 1.27)) hide)
+    )
+    (property "Datasheet" "http://www.vishay.com/docs/88503/1n4001.pdf" (at 92.71 87.63 0)
+      (effects (font (size 1.27 1.27)) hide)
+    )
+    (property "Sim.Device" "D" (at 92.71 87.63 0)
+      (effects (font (size 1.27 1.27)) hide)
+    )
+    (property "Sim.Pins" "1=K 2=A" (at 92.71 87.63 0)
+      (effects (font (size 1.27 1.27)) hide)
+    )
+    (pin "2")
+    (pin "1")
+    (instances
+      (project "BatterySource-Kicad"
+        (path "/95ddd1e1-59e3-4dac-b83b-1bbc0d6327ef"
+          (reference "D1") (unit 1)
+        )
+      )
+    )
+  )
+  (symbol (lib_id "Device:R") (at 92.71 54.61 0) (unit 1)
+    (in_bom yes) (on_board yes) (dnp no) (fields_autoplaced)
+    (property "Reference" "R1" (at 95.25 53.34 0)
+      (effects (font (size 1.27 1.27)) (justify left))
+    )
+    (property "Value" "1k" (at 95.25 55.88 0)
+      (effects (font (size 1.27 1.27)) (justify left))
+    )
+    (property "Footprint" "" (at 90.932 54.61 90)
+      (effects (font (size 1.27 1.27)) hide)
+    )
+    (property "Datasheet" "~" (at 92.71 54.61 0)
+      (effects (font (size 1.27 1.27)) hide)
+    )
+    (pin "1")
+    (pin "2")
+    (instances
+      (project "BatterySource-Kicad"
+        (path "/95ddd1e1-59e3-4dac-b83b-1bbc0d6327ef"
+          (reference "R1") (unit 1)
+        )
+      )
+    )
+  )
+  (symbol (lib_id "Diode:1N4007") (at 92.71 80.01 90) (unit 1)
+    (in_bom yes) (on_board yes) (dnp no) (fields_autoplaced)
+    (property "Reference" "D2" (at 95.25 78.74 90)
+      (effects (font (size 1.27 1.27)) (justify right))
+    )
+    (property "Value" "1N4007" (at 95.25 81.28 90)
+      (effects (font (size 1.27 1.27)) (justify right))
+    )
+    (property "Footprint" "Diode_THT:D_DO-41_SOD81_P10.16mm_Horizontal" (at 97.155 80.01 0)
+      (effects (font (size 1.27 1.27)) hide)
+    )
+    (property "Datasheet" "http://www.vishay.com/docs/88503/1n4001.pdf" (at 92.71 80.01 0)
+      (effects (font (size 1.27 1.27)) hide)
+    )
+    (property "Sim.Device" "D" (at 92.71 80.01 0)
+      (effects (font (size 1.27 1.27)) hide)
+    )
+    (property "Sim.Pins" "1=K 2=A" (at 92.71 80.01 0)
+      (effects (font (size 1.27 1.27)) hide)
+    )
+    (pin "2")
+    (pin "1")
+    (instances
+      (project "BatterySource-Kicad"
+        (path "/95ddd1e1-59e3-4dac-b83b-1bbc0d6327ef"
+          (reference "D2") (unit 1)
+        )
+      )
+    )
+  )
+  (symbol (lib_id "power:+12V") (at 92.71 40.64 0) (unit 1)
+    (in_bom yes) (on_board yes) (dnp no) (fields_autoplaced)
+    (property "Reference" "#PWR01" (at 92.71 44.45 0)
+      (effects (font (size 1.27 1.27)) hide)
+    )
+    (property "Value" "+12V" (at 92.71 35.56 0)
+      (effects (font (size 1.27 1.27)))
+    )
+    (property "Footprint" "" (at 92.71 40.64 0)
+      (effects (font (size 1.27 1.27)) hide)
+    )
+    (property "Datasheet" "" (at 92.71 40.64 0)
+      (effects (font (size 1.27 1.27)) hide)
+    )
+    (pin "1")
+    (instances
+      (project "BatterySource-Kicad"
+        (path "/95ddd1e1-59e3-4dac-b83b-1bbc0d6327ef"
+          (reference "#PWR01") (unit 1)
+        )
+      )
+    )
+  )
+  (symbol (lib_id "Diode:1N4007") (at 92.71 72.39 90) (unit 1)
+    (in_bom yes) (on_board yes) (dnp no) (fields_autoplaced)
+    (property "Reference" "D3" (at 95.25 71.12 90)
+      (effects (font (size 1.27 1.27)) (justify right))
+    )
+    (property "Value" "1N4007" (at 95.25 73.66 90)
+      (effects (font (size 1.27 1.27)) (justify right))
+    )
+    (property "Footprint" "Diode_THT:D_DO-41_SOD81_P10.16mm_Horizontal" (at 97.155 72.39 0)
+      (effects (font (size 1.27 1.27)) hide)
+    )
+    (property "Datasheet" "http://www.vishay.com/docs/88503/1n4001.pdf" (at 92.71 72.39 0)
+      (effects (font (size 1.27 1.27)) hide)
+    )
+    (property "Sim.Device" "D" (at 92.71 72.39 0)
+      (effects (font (size 1.27 1.27)) hide)
+    )
+    (property "Sim.Pins" "1=K 2=A" (at 92.71 72.39 0)
+      (effects (font (size 1.27 1.27)) hide)
+    )
+    (pin "2")
+    (pin "1")
+    (instances
+      (project "BatterySource-Kicad"
+        (path "/95ddd1e1-59e3-4dac-b83b-1bbc0d6327ef"
+          (reference "D3") (unit 1)
+        )
+      )
+    )
+  )
+  (symbol (lib_id "power:GND") (at 92.71 100.33 0) (unit 1)
+    (in_bom yes) (on_board yes) (dnp no) (fields_autoplaced)
+    (property "Reference" "#PWR02" (at 92.71 106.68 0)
+      (effects (font (size 1.27 1.27)) hide)
+    )
+    (property "Value" "GND" (at 92.71 105.41 0)
+      (effects (font (size 1.27 1.27)))
+    )
+    (property "Footprint" "" (at 92.71 100.33 0)
+      (effects (font (size 1.27 1.27)) hide)
+    )
+    (property "Datasheet" "" (at 92.71 100.33 0)
+      (effects (font (size 1.27 1.27)) hide)
+    )
+    (pin "1")
+    (instances
+      (project "BatterySource-Kicad"
+        (path "/95ddd1e1-59e3-4dac-b83b-1bbc0d6327ef"
+          (reference "#PWR02") (unit 1)
+        )
+      )
+    )
+  )
+  (sheet_instances
+    (path "/" (page "1"))
+  )
 )

Commit message: Finished circuit Kicad
Parts:
- added C1: 1u, symbol Device:C_Polarized
- added D4: LED, symbol Device:LED
- added D5, D6, D7: 1N4007, Diode_THT:D_DO-41_SOD81_P10.16mm_Horizontal, symbol Diode:1N4007
- added Q1, Q2: NPN, symbol Simulation_SPICE:NPN
- added R2: 550, symbol Device:R
- added R3: 100k, symbol Device:R
- added R4: 220, symbol Device:R
- added RV1, RV2: 10k, symbol Device:R_Potentiometer
- added U1: RC4558, symbol Amplifier_Operational:RC4558
- R1: value 1k -> 100k
Connections:
- net +12V: now also C1.1, Q1.1 (C), Q2.1 (C), R3.1, RV1.1, U1.8 (V+)
- net GND: now also C1.2, D4.1 (K), D7.1 (K), RV1.3, RV2.3, U1.4 (V-)
- net at D3.2 (A), R1.2: now also U1.3 (+)
- new net: Q2.2 (B), U1.1
- new net: Q2.3 (E), R2.1
- new net: D5.2 (A), R3.2, U1.5 (+)
- new net: D5.1 (K), D6.2 (A)
- new net: Q1.3 (E), RV2.1
- new net: RV2.2, U1.6 (-)
- new net: Q1.2 (B), R4.1
- new net: R4.2, U1.7
- new net: D4.2 (A), R2.2
- new net: D6.1 (K), D7.2 (A)
- new net: RV1.2, U1.2 (-)
Other:
- moved on the sheet: D1, D2, D3, R1

Commit message: Finished schematic and strip layout
Parts:
- added C2: 1u, symbol Device:C_Polarized
- added J1: IN/BATT, symbol Connector:Screw_Terminal_01x02
- added J2: OUT, symbol Connector:Screw_Terminal_01x02
- Q1, Q2: value NPN -> NPN - 2SD882
- R4: value 220 -> 550
Connections:
- net +12V: now also J1.1 (Pin_1)
- net GND: now also C2.2, J1.2 (Pin_2), J2.2 (Pin_2)
- net at Q1.3 (E), RV2.1: now also C2.1, J2.1 (Pin_1)
Changed lines of the file:
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@@
   (junction (at 129.54 95.25) (diameter 0) (color 0 0 0 0)
   )
+  (junction (at 201.93 45.72) (diameter 0) (color 0 0 0 0)
+  )
   (junction (at 31.75 33.02) (diameter 0) (color 0 0 0 0)
   )
+  (junction (at 214.63 95.25) (diameter 0) (color 0 0 0 0)
+  )
+  (junction (at 201.93 95.25) (diameter 0) (color 0 0 0 0)
+  )
   (junction (at 152.4 45.72) (diameter 0) (color 0 0 0 0)
   )
@@
   (junction (at 92.71 95.25) (diameter 0) (color 0 0 0 0)
   )
+  (junction (at 214.63 45.72) (diameter 0) (color 0 0 0 0)
+  )
   (junction (at 31.75 53.34) (diameter 0) (color 0 0 0 0)
   )
@@
     (stroke (width 0) (type default))
   )
+  (wire (pts (xy 49.53 53.34) (xy 31.75 53.34))
+    (stroke (width 0) (type default))
+  )
   (wire (pts (xy 81.28 40.64) (xy 81.28 45.72))
     (stroke (width 0) (type default))
@@
     (stroke (width 0) (type default))
   )
+  (wire (pts (xy 49.53 44.45) (xy 49.53 53.34))
+    (stroke (width 0) (type default))
+  )
   (wire (pts (xy 21.59 40.64) (xy 21.59 33.02))
     (stroke (width 0) (type default))
   )
+  (wire (pts (xy 214.63 76.2) (xy 214.63 95.25))
+    (stroke (width 0) (type default))
+  )
+  (wire (pts (xy 214.63 68.58) (xy 214.63 45.72))
+    (stroke (width 0) (type default))
+  )
   (wire (pts (xy 81.28 57.15) (xy 81.28 60.96))
     (stroke (width 0) (type default))
@@
     (stroke (width 0) (type default))
   )
+  (wire (pts (xy 227.33 95.25) (xy 214.63 95.25))
+    (stroke (width 0) (type default))
+  )
   (wire (pts (xy 31.75 53.34) (xy 31.75 58.42))
     (stroke (width 0) (type default))
@@
     (stroke (width 0) (type default))
   )
+  (wire (pts (xy 214.63 45.72) (xy 227.33 45.72))
+    (stroke (width 0) (type default))
+  )
   (wire (pts (xy 129.54 95.25) (xy 152.4 95.25))
     (stroke (width 0) (type default))
@@
     (stroke (width 0) (type default))
   )
+  (wire (pts (xy 49.53 41.91) (xy 49.53 33.02))
+    (stroke (width 0) (type default))
+  )
   (wire (pts (xy 21.59 48.26) (xy 21.59 53.34))
     (stroke (width 0) (type default))
   )
+  (wire (pts (xy 214.63 45.72) (xy 201.93 45.72))
+    (stroke (width 0) (type default))
+  )
   (wire (pts (xy 201.93 45.72) (xy 195.58 45.72))
     (stroke (width 0) (type default))
   )
+  (wire (pts (xy 227.33 48.26) (xy 227.33 95.25))
+    (stroke (width 0) (type default))
+  )
   (wire (pts (xy 129.54 45.72) (xy 92.71 45.72))
     (stroke (width 0) (type default))
@@
     (stroke (width 0) (type default))
   )
+  (wire (pts (xy 49.53 33.02) (xy 31.75 33.02))
+    (stroke (width 0) (type default))
+  )
   (wire (pts (xy 152.4 45.72) (xy 185.42 45.72))
     (stroke (width 0) (type default))
   )
   (wire (pts (xy 81.28 60.96) (xy 81.28 68.58))
+    (stroke (width 0) (type default))
+  )
+  (wire (pts (xy 214.63 95.25) (xy 201.93 95.25))
     (stroke (width 0) (type default))
   )
@@
       (effects (font (size 1.27 1.27)) (justify left))
     )
-    (property "Value" "NPN" (at 132.08 64.77 0)
+    (property "Value" "NPN - 2SD882" (at 132.08 64.77 0)
       (effects (font (size 1.27 1.27)) (justify left))
     )
@@
         (path "/95ddd1e1-59e3-4dac-b83b-1bbc0d6327ef"
           (reference "R3") (unit 1)
+        )
+      )
+    )
+  )
+  (symbol (lib_id "Connector:Screw_Terminal_01x02") (at 232.41 45.72 0) (unit 1)
+    (in_bom yes) (on_board yes) (dnp no) (fields_autoplaced)
+    (property "Reference" "J2" (at 234.95 45.72 0)
+      (effects (font (size 1.27 1.27)) (justify left))
+    )
+    (property "Value" "OUT" (at 234.95 48.26 0)
+      (effects (font (size 1.27 1.27)) (justify left))
+    )
+    (property "Footprint" "" (at 232.41 45.72 0)
+      (effects (font (size 1.27 1.27)) hide)
+    )
+    (property "Datasheet" "~" (at 232.41 45.72 0)
+      (effects (font (size 1.27 1.27)) hide)
+    )
+    (pin "1")
+    (pin "2")
+    (instances
+      (project "BatterySource-Kicad"
+        (path "/95ddd1e1-59e3-4dac-b83b-1bbc0d6327ef"
+          (reference "J2") (unit 1)
         )
       )
@@
       (effects (font (size 1.27 1.27)) (justify left))
     )
-    (property "Value" "220" (at 193.04 60.96 0)
+    (property "Value" "550" (at 193.04 60.96 0)
       (effects (font (size 1.27 1.27)) (justify left))
     )
@@
       (effects (font (size 1.27 1.27)))
     )
-    (property "Value" "NPN" (at 190.5 41.91 90)
+    (property "Value" "NPN - 2SD882" (at 190.5 41.91 90)
       (effects (font (size 1.27 1.27)))
     )
@@
     )
   )
+  (symbol (lib_id "Device:C_Polarized") (at 214.63 72.39 0) (unit 1)
+    (in_bom yes) (on_board yes) (dnp no) (fields_autoplaced)
+    (property "Reference" "C2" (at 218.44 70.231 0)
+      (effects (font (size 1.27 1.27)) (justify left))
+    )
+    (property "Value" "1u" (at 218.44 72.771 0)
+      (effects (font (size 1.27 1.27)) (justify left))
+    )
+    (property "Footprint" "" (at 215.5952 76.2 0)
+      (effects (font (size 1.27 1.27)) hide)
+    )
+    (property "Datasheet" "~" (at 214.63 72.39 0)
+      (effects (font (size 1.27 1.27)) hide)
+    )
+    (pin "1")
+    (pin "2")
+    (instances
+      (project "BatterySource-Kicad"
+        (path "/95ddd1e1-59e3-4dac-b83b-1bbc0d6327ef"
+          (reference "C2") (unit 1)
+        )
+      )
+    )
+  )
   (symbol (lib_id "Device:R_Potentiometer") (at 92.71 74.93 0) (unit 1)
     (in_bom yes) (on_board yes) (dnp no) (fields_autoplaced)
@@
         )
       )
+    )
+  )
+  (symbol (lib_id "Connector:Screw_Terminal_01x02") (at 54.61 41.91 0) (unit 1)
+    (in_bom yes) (on_board yes) (dnp no) (fields_autoplaced)
+    (property "Reference" "J1" (at 57.15 41.91 0)
+      (effects (font (size 1.27 1.27)) (justify left))
+    )
+    (property "Value" "IN/BATT" (at 57.15 44.45 0)
+      (effects (font (size 1.27 1.27)) (justify left))
+    )
+    (property "Footprint" "" (at 54.61 41.91 0)
+      (effects (font (size 1.27 1.27)) hide)
+    )
+    (property "Datasheet" "~" (at 54.61 41.91 0)
+      (effects (font (size 1.27 1.27)) hide)
+    )
+    (pin "1")
+    (pin "2")
+    (instances
+      (project "BatterySource-Kicad"
+        (path "/95ddd1e1-59e3-4dac-b83b-1bbc0d6327ef"
+          (reference "J1") (unit 1)
+        )
+      )

Commit message: Added on/off switch and LED to kicad schematic and stripboard layout
Finished and it works (does not match prototype)
Parts:
- added D8: LED, symbol Device:LED
- added R5: 550, symbol Device:R
- added SW1: SW_SPST, symbol Switch:SW_SPST
Connections:
- net +12V: now also R5.1, SW1.2 (B); no longer J1.1 (Pin_1)
- net GND: now also D8.1 (K)
- new net: D8.2 (A), R5.2
- new net: J1.1 (Pin_1), SW1.1 (A)
Other:
- moved on the sheet: C1, C2, D1, D2, D3, D4, D5, D6, D7, J1, J2, Q1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
